Commit message: Setup camera + correction setup v2

File: src/motoman/motoman_hc10_support/urdf/hc10_control.xacro (robot description, xacro)
@@ -15,5 +15,4 @@
             </transmission>
         </xacro:macro>
-        <xacro:hc10_arm_control transmission="${prefix}_tran_base" joint="${prefix}world_fixed" motor="${prefix}_motor_base"/>
         <xacro:hc10_arm_control transmission="${prefix}_tran_1" joint="${prefix}joint_1_s" motor="${prefix}_motor_1"/>
         <xacro:hc10_arm_control transmission="${prefix}_tran_2" joint="${prefix}joint_2_l" motor="${prefix}_motor_2"/>

File: src/motoman/motoman_hc10_support/urdf/hc10_gazebo_macro.xacro (robot description, xacro)
@@ -17,11 +17,4 @@
             </gazebo>
         </xacro:macro>
-        <xacro:macro name="hc10_hand_gazebo" params="link">
-            <gazebo reference="${link}">
-                <material>Gazebo/Grey</material>
-                <mu1>0.2</mu1>
-                <mu2>0.2</mu2>
-            </gazebo>
-        </xacro:macro>
         <xacro:hc10_env link="${prefix}box_fixed"/>
         <xacro:hc10_arm link="${prefix}base_link"/>
@@ -31,7 +24,7 @@
         <xacro:hc10_arm link="${prefix}link_4_r"/>
         <xacro:hc10_arm link="${prefix}link_5_b"/>
-        <xacro:hc10_hand_gazebo link="${prefix}link_6_t"/>
-        <xacro:hc10_hand_gazebo link="${prefix}tool0"/>
-        <xacro:hc10_hand_gazebo link="${prefix}camera_link"/>
+        <xacro:hc10_arm link="${prefix}link_6_t"/>
+        <xacro:hc10_arm link="${prefix}tool0"/>
+        <xacro:hc10_arm link="${prefix}camera_link"/>
     </xacro:macro>
 </robot>
