Commit message: delete submodule

File: src/motoman/motoman_hc10_support/urdf/hc10_macro.xacro (robot description, xacro)
@@ -5,4 +5,8 @@
     <!-- link list -->
     <link name="world"/>
+    <joint name="world_fixed" type="fixed">
+      <parent link="world"/>
+      <child link="${prefix}base_link"/>
+    </joint>
     <link name="${prefix}base_link">
       <inertial>
@@ -134,8 +138,4 @@
     <!-- end of link list -->
     <!-- joint list -->
-    <joint name="world_fixed" type="fixed">
-      <parent link="world"/>
-      <child link="${prefix}base_link"/>
-    </joint>
     <joint name="${prefix}joint_1_s" type="revolute">
       <parent link="${prefix}base_link"/>

Commit message: init push

File: src/motoman/motoman_hc10_support/urdf/hc10_macro.xacro (robot description, xacro)
@@ -5,137 +5,137 @@
     <!-- link list -->
     <link name="world"/>
+    <link name="${prefix}base_link">
+      <inertial>
+        <origin xyz="0 0 0" rpy="0 0 0"/>
+        <mass value="0.1"/>
+        <inertia ixx="0.03" ixy="0.03" ixz="0.03" iyy="0.0" iyz="0.0" izz="0.0"/>
+      </inertial>
+      <visual>
+        <geometry>
+          <mesh filename="package://motoman_hc10_support/meshes/hc10/visual/base_link.dae"/>
+        </geometry>
+        <xacro:material_yaskawa_blue/>
+      </visual>
+      <collision>
+        <geometry>
+          <mesh filename="package://motoman_hc10_support/meshes/hc10/collision/base_link.stl"/>
+        </geometry>
+      </collision>
+    </link>
+    <link name="${prefix}link_1_s">
+      <inertial>
+        <origin xyz="0 0 0" rpy="0 0 0"/>
+        <mass value="0.1"/>
+        <inertia ixx="0.03" ixy="0.03" ixz="0.03" iyy="0.0" iyz="0.0" izz="0.0"/>
+      </inertial>
+      <visual>
+        <geometry>
+          <mesh filename="package://motoman_hc10_support/meshes/hc10/visual/link_1_s.dae"/>
+        </geometry>
+        <xacro:material_yaskawa_blue/>
+      </visual>
+      <collision>
+        <geometry>
+          <mesh filename="package://motoman_hc10_support/meshes/hc10/collision/link_1_s.stl"/>
+        </geometry>
+      </collision>
+    </link>
+    <link name="${prefix}link_2_l">
+      <inertial>
+        <origin xyz="0 0 0" rpy="0 0 0"/>
+        <mass value="0.1"/>
+        <inertia ixx="0.03" ixy="0.03" ixz="0.03" iyy="0.0" iyz="0.0" izz="0.0"/>
+      </inertial>
+      <visual>
+        <geometry>
+          <mesh filename="package://motoman_hc10_support/meshes/hc10/visual/link_2_l.dae"/>
+        </geometry>
+        <xacro:material_yaskawa_blue/>
+      </visual>
+      <collision>
+        <geometry>
+          <mesh filename="package://motoman_hc10_support/meshes/hc10/collision/link_2_l.stl"/>
+        </geometry>
+      </collision>hc10_macro
+    </link>
+    <link name="${prefix}link_3_u">
+      <inertial>
+        <origin xyz="0 0 0" rpy="0 0 0"/>
+        <mass value="0.1"/>
+        <inertia ixx="0.03" ixy="0.03" ixz="0.03" iyy="0.0" iyz="0.0" izz="0.0"/>
+      </inertial>
+      <visual>
+        <geometry>
+          <mesh filename="package://motoman_hc10_support/meshes/hc10/visual/link_3_u.dae"/>
+        </geometry>
+        <xacro:material_yaskawa_blue/>
+      </visual>
+      <collision>
+        <geometry>
+          <mesh filename="package://motoman_hc10_support/meshes/hc10/collision/link_3_u.stl"/>
+        </geometry>
+      </collision>
+    </link>
+    <link name="${prefix}link_4_r">
+      <inertial>
+        <origin xyz="0 0 0" rpy="0 0 0"/>
+        <mass value="0.1"/>
+        <inertia ixx="0.03" ixy="0.03" ixz="0.03" iyy="0.0" iyz="0.0" izz="0.0"/>
+      </inertial>
+      <visual>
+        <geometry>
+          <mesh filename="package://motoman_hc10_support/meshes/hc10/visual/link_4_r.dae"/>
+        </geometry>
+        <xacro:material_yaskawa_blue/>
+      </visual>
+      <collision>
+        <geometry>
+          <mesh filename="package://motoman_hc10_support/meshes/hc10/collision/link_4_r.stl"/>
+        </geometry>
+      </collision>
+    </link>
+    <link name="${prefix}link_5_b">
+      <inertial>
+        <origin xyz="0 0 0" rpy="0 0 0"/>
+        <mass value="0.1"/>
+        <inertia ixx="0.03" ixy="0.03" ixz="0.03" iyy="0.0" iyz="0.0" izz="0.0"/>
+      </inertial>
+      <visual>
+        <geometry>
+          <mesh filename="package://motoman_hc10_support/meshes/hc10/visual/link_5_b.dae"/>
+        </geometry>
+        <xacro:material_yaskawa_blue/>
+      </visual>
+      <collision>
+        <geometry>
+          <mesh filename="package://motoman_hc10_support/meshes/hc10/collision/link_5_b.stl"/>
+        </geometry>
+      </collision>
+    </link>
+    <link name="${prefix}link_6_t">
+      <inertial>
+        <origin xyz="0 0 0" rpy="0 0 0"/>
+        <mass value="0.1"/>
+        <inertia ixx="0.03" ixy="0.03" ixz="0.03" iyy="0.0" iyz="0.0" izz="0.0"/>
+      </inertial>
+      <visual>
+        <geometry>
+          <mesh filename="package://motoman_hc10_support/meshes/hc10/visual/link_6_t.dae"/>
+        </geometry>
+        <xacro:material_yaskawa_blue/>
+      </visual>
+      <collision>
+        <geometry>
+          <mesh filename="package://motoman_hc10_support/meshes/hc10/collision/link_6_t.stl"/>
+        </geometry>
+      </collision>
+    </link>
+    <link name="${prefix}tool0"/>
+    <!-- end of link list -->
+    <!-- joint list -->
     <joint name="world_fixed" type="fixed">
       <parent link="world"/>
       <child link="${prefix}base_link"/>
     </joint>
-    <link name="${prefix}base_link">
-      <inertial>
-        <origin xyz="0 0 0" rpy="0 0 0"/>
-        <mass value="0.1"/>
-        <inertia ixx="0.03" ixy="0.03" ixz="0.03" iyy="0.0" iyz="0.0" izz="0.0"/>
-      </inertial>
-      <visual>
-        <geometry>
-          <mesh filename="package://motoman_hc10_support/meshes/hc10/visual/base_link.dae"/>
-        </geometry>
-        <xacro:material_yaskawa_blue/>
-      </visual>
-      <collision>
-        <geometry>
-          <mesh filename="package://motoman_hc10_support/meshes/hc10/collision/base_link.stl"/>
-        </geometry>
-      </collision>
-    </link>
-    <link name="${prefix}link_1_s">
-      <inertial>
-        <origin xyz="0 0 0" rpy="0 0 0"/>
-        <mass value="0.1"/>
-        <inertia ixx="0.03" ixy="0.03" ixz="0.03" iyy="0.0" iyz="0.0" izz="0.0"/>
-      </inertial>
-      <visual>
-        <geometry>
-          <mesh filename="package://motoman_hc10_support/meshes/hc10/visual/link_1_s.dae"/>
-        </geometry>
-        <xacro:material_yaskawa_blue/>
-      </visual>
-      <collision>
-        <geometry>
-          <mesh filename="package://motoman_hc10_support/meshes/hc10/collision/link_1_s.stl"/>
-        </geometry>
-      </collision>
-    </link>
-    <link name="${prefix}link_2_l">
-      <inertial>
-        <origin xyz="0 0 0" rpy="0 0 0"/>
-        <mass value="0.1"/>
-        <inertia ixx="0.03" ixy="0.03" ixz="0.03" iyy="0.0" iyz="0.0" izz="0.0"/>
-      </inertial>
-      <visual>
-        <geometry>
-          <mesh filename="package://motoman_hc10_support/meshes/hc10/visual/link_2_l.dae"/>
-        </geometry>
-        <xacro:material_yaskawa_blue/>
-      </visual>
-      <collision>
-        <geometry>
-          <mesh filename="package://motoman_hc10_support/meshes/hc10/collision/link_2_l.stl"/>
-        </geometry>
-      </collision>hc10_macro
-    </link>
-    <link name="${prefix}link_3_u">
-      <inertial>
-        <origin xyz="0 0 0" rpy="0 0 0"/>
-        <mass value="0.1"/>
-        <inertia ixx="0.03" ixy="0.03" ixz="0.03" iyy="0.0" iyz="0.0" izz="0.0"/>
-      </inertial>
-      <visual>
-        <geometry>
-          <mesh filename="package://motoman_hc10_support/meshes/hc10/visual/link_3_u.dae"/>
-        </geometry>
-        <xacro:material_yaskawa_blue/>
-      </visual>
-      <collision>
-        <geometry>
-          <mesh filename="package://motoman_hc10_support/meshes/hc10/collision/link_3_u.stl"/>
-        </geometry>
-      </collision>
-    </link>
-    <link name="${prefix}link_4_r">
-      <inertial>
-        <origin xyz="0 0 0" rpy="0 0 0"/>
-        <mass value="0.1"/>
-        <inertia ixx="0.03" ixy="0.03" ixz="0.03" iyy="0.0" iyz="0.0" izz="0.0"/>
-      </inertial>
-      <visual>
-        <geometry>
-          <mesh filename="package://motoman_hc10_support/meshes/hc10/visual/link_4_r.dae"/>
-        </geometry>
-        <xacro:material_yaskawa_blue/>
-      </visual>
-      <collision>
-        <geometry>
-          <mesh filename="package://motoman_hc10_support/meshes/hc10/collision/link_4_r.stl"/>
-        </geometry>
-      </collision>
-    </link>
-    <link name="${prefix}link_5_b">
-      <inertial>
-        <origin xyz="0 0 0" rpy="0 0 0"/>
-        <mass value="0.1"/>
-        <inertia ixx="0.03" ixy="0.03" ixz="0.03" iyy="0.0" iyz="0.0" izz="0.0"/>
-      </inertial>
-      <visual>
-        <geometry>
-          <mesh filename="package://motoman_hc10_support/meshes/hc10/visual/link_5_b.dae"/>
-        </geometry>
-        <xacro:material_yaskawa_blue/>
-      </visual>
-      <collision>
-        <geometry>
-          <mesh filename="package://motoman_hc10_support/meshes/hc10/collision/link_5_b.stl"/>
-        </geometry>
-      </collision>
-    </link>
-    <link name="${prefix}link_6_t">
-      <inertial>
-        <origin xyz="0 0 0" rpy="0 0 0"/>
-        <mass value="0.1"/>
-        <inertia ixx="0.03" ixy="0.03" ixz="0.03" iyy="0.0" iyz="0.0" izz="0.0"/>
-      </inertial>
-      <visual>
-        <geometry>
-          <mesh filename="package://motoman_hc10_support/meshes/hc10/visual/link_6_t.dae"/>
-        </geometry>
-        <xacro:material_yaskawa_blue/>
-      </visual>
-      <collision>
-        <geometry>
-          <mesh filename="package://motoman_hc10_support/meshes/hc10/collision/link_6_t.stl"/>
-        </geometry>
-      </collision>
-    </link>
-    <link name="${prefix}tool0"/>
-    <!-- end of link list -->
-    <!-- joint list -->
     <joint name="${prefix}joint_1_s" type="revolute">
       <parent link="${prefix}base_link"/>

Commit message: Setup camera + correction setup v3

File: src/motoman/motoman_hc10_support/urdf/hc10_macro.xacro (robot description, xacro)
@@ -194,10 +194,4 @@
     <!-- end of joint list -->
     <!-- ROS base_link to Robot Manufacturer World Coordinates transform -->
-    <link name="${prefix}base" />
-    <joint name="${prefix}base_link-base" type="fixed">
-      <origin xyz="0 0 0.275" rpy="0 0 0"/>
-      <parent link="${prefix}base_link"/>
-      <child link="${prefix}base"/>
-    </joint>
   </xacro:macro>
 </robot>

File: src/motoman/motoman_hc10_support/urdf/hc10_sensor.xacro (robot description, xacro)
@@ -17,5 +17,4 @@
    	  <box size="0.010 0.03 0.03"/>
   	</geometry>
-   	<material name="red"/>
      </visual>
    </link>
