Commit message: completed env

File: src/motoman/motoman_hc10_support/urdf/hc10_env_macro.xacro (robot description, xacro)
@@ -1,36 +1,115 @@
 <?xml version='1.0' encoding='utf-8'?>
-<!-- panda.gazebo.xacro -->
 <robot xmlns:xacro="http://www.ros.org/wiki/xacro">
     <xacro:macro name="hc10_workspace" params="prefix">
+        <!-- Définir le socle -->
         <link name="box">
             <visual>
-              <origin xyz="0 0 0" rpy="0 0 0"/>
-              <geometry>
-                <box size="1.5 1.5 0.15"/>
-             </geometry>
-              <material name="blue">
-                <color rgba="0 0 0.8 1"/>
-              </material>
+                <origin xyz="0 0 0" rpy="0 0 0"/>
+                <geometry>
+                    <box size="1.5 1.5 0.15"/>
+                </geometry>
+                <material name="blue">
+                    <color rgba="0 0 0.8 1"/>
+                </material>
             </visual>
             <collision>
-              <origin xyz="0 0 0" rpy="0 0 0"/>
-              <geometry>
-                <box size="1.5 1.5 0.15"/>
-              </geometry>
+                <origin xyz="0 0 0" rpy="0 0 0"/>
+                <geometry>
+                    <box size="1.5 1.5 0.15"/>
+                </geometry>
             </collision>
             <inertial>
-              <origin xyz="0 0 0" rpy="0 0 0"/>
-              <mass value="100"/>
-              <inertia ixx="1" ixy="0" ixz="0" iyy="1" iyz="0" izz="1"/>
+                <origin xyz="0 0 0" rpy="0 0 0"/>
+                <mass value="100"/>
+                <inertia ixx="1" ixy="0" ixz="0" iyy="1" iyz="0" izz="1"/>
             </inertial>
         </link>
-        <!-- joint list -->
+        <!-- Ajouter les parois  -->
+        <link name="wall1">
+            <visual>
+                <origin xyz="0 0.7 0.825" rpy="0 0 0"/>
+                <geometry>
+                    <box size="1.3 0.1 1.5"/>
+                </geometry>
+                <material name="glass">
+                    <color rgba="0.8 0.8 0.8 0.5"/> <!-- Couleur transparente pour du verre -->
+                </material>
+            </visual>
+            <collision>
+                <origin xyz="0 0.7 0.825" rpy="0 0 0"/>
+                <geometry>
+                    <box size="1.5 0.1 1.5"/>
+                </geometry>
+            </collision>
+            <inertial>
+                <origin xyz="0 0.7 0.825" rpy="0 0 0"/>
+                <mass value="1"/>
+                <inertia ixx="1" ixy="0" ixz="0" iyy="1" iyz="0" izz="1"/>
+            </inertial>
+        </link>
+        <link name="wall2">
+            <visual>
+                <origin xyz="-0.7 0 0.825" rpy="0 0 0"/>
+                <geometry>
+                    <box size="0.1 1.5 1.5"/>
+                </geometry>
+                <material name="glass">
+                    <color rgba="0.8 0.8 0.8 0.5"/> <!-- Couleur transparente pour du verre -->
+                </material>
+            </visual>
+            <collision>
+                <origin xyz="-0.7 0 0.825" rpy="0 0 0"/>
+                <geometry>
+                    <box size="0.1 1.5 1.5"/>
+                </geometry>
+            </collision>
+            <inertial>
+                <origin xyz="-0.7 0 0.825" rpy="0 0 0"/>
+                <mass value="1"/>
+                <inertia ixx="1" ixy="0" ixz="0" iyy="1" iyz="0" izz="1"/>
+            </inertial>
+        </link>
+        <link name="wall3">
+            <visual>
+                <origin xyz="0.7 0 0.825" rpy="0 0 0"/>
+                <geometry>
+                    <box size="0.1 1.5 1.5"/>
+                </geometry>
+                <material name="glass">
+                    <color rgba="0.8 0.8 0.8 0.5"/> <!-- Couleur transparente pour du verre -->
+                </material>
+            </visual>
+            <collision>
+                <origin xyz="0.7 0 0.825" rpy="0 0 0"/>
+                <geometry>
+                    <box size="0.1 1.5 1.5"/>
+                </geometry>
+            </collision>
+            <inertial>
+                <origin xyz="0.7 0 0.825" rpy="0 0 0"/>
+                <mass value="1"/>
+                <inertia ixx="1" ixy="0" ixz="0" iyy="1" iyz="0" izz="1"/>
+            </inertial>
+        </link>
+        <!-- joint list pour le socle -->
         <joint name="box_fixed" type="revolute">
             <parent link="world"/>
-            <child link="${prefix}box"/>
+            <child link="box"/>
             <origin xyz="0.75 0.75 0.075" rpy="0 0 0" />
             <dynamics damping="1"/>
             <limit lower="-3.14159" upper="3.14159" effort="10.0" velocity="0.5"/>
         </joint>
+        <joint name="wall1_fixed" type="fixed">
+            <parent link="box"/>
+            <child link="wall1"/>
+        </joint>
+        <joint name="wall2_fixed" type="fixed">
+            <parent link="box"/>
+            <child link="wall2"/>
+        </joint>
+        <joint name="wall3_fixed" type="fixed">
+            <parent link="box"/>
+            <child link="wall3"/>
+        </joint>
     </xacro:macro>
 </robot>

File: src/motoman/motoman_hc10_support/urdf/hc10_gazebo_macro.xacro (robot description, xacro)
@@ -25,4 +25,7 @@
         </xacro:macro>
         <xacro:hc10_env link="${prefix}box_fixed"/>
+        <xacro:hc10_env link="${prefix}wall1"/>
+        <xacro:hc10_env link="${prefix}wall2"/>
+        <xacro:hc10_env link="${prefix}wall3"/>
         <xacro:hc10_arm link="${prefix}base_link"/>
         <xacro:hc10_arm link="${prefix}link_1_s"/>

File: src/motoman/motoman_hc10_support/urdf/hc10_macro.xacro (robot description, xacro)
@@ -137,5 +137,5 @@
       <parent link="world"/>
       <child link="${prefix}base_link"/>
-      <origin xyz="0.1 0.1 0.5" rpy="0 0 0" />
+      <origin xyz="0.55 0.4 0.15" rpy="0 0 0" />
     </joint>
     <joint name="${prefix}joint_1_s" type="revolute">

Commit message: corrected environment components

File: src/motoman/motoman_hc10_support/urdf/hc10_env_macro.xacro (robot description, xacro)
@@ -5,5 +5,5 @@
         <link name="box">
             <visual>
-                <origin xyz="0 0 0" rpy="0 0 0"/>
+                <origin xyz="0.75 0.75 0.075" rpy="0 0 0"/>
                 <geometry>
                     <box size="1.5 1.5 0.15"/>
@@ -14,5 +14,5 @@
             </visual>
             <collision>
-                <origin xyz="0 0 0" rpy="0 0 0"/>
+                <origin xyz="0.75 0.75 0.075" rpy="0 0 0"/>
                 <geometry>
                     <box size="1.5 1.5 0.15"/>
@@ -20,5 +20,5 @@
             </collision>
             <inertial>
-                <origin xyz="0 0 0" rpy="0 0 0"/>
+                <origin xyz="0.75 0.75 0.075" rpy="0 0 0"/>
                 <mass value="100"/>
                 <inertia ixx="1" ixy="0" ixz="0" iyy="1" iyz="0" izz="1"/>
@@ -26,7 +26,7 @@
         </link>
         <!-- Ajouter les parois  -->
-        <link name="wall1">
+        <link name="wall_fond">
             <visual>
-                <origin xyz="0 0.7 0.825" rpy="0 0 0"/>
+                <origin xyz="0.75 1.45 0.9" rpy="0 0 0"/>
                 <geometry>
                     <box size="1.3 0.1 1.5"/>
@@ -37,5 +37,5 @@
             </visual>
             <collision>
-                <origin xyz="0 0.7 0.825" rpy="0 0 0"/>
+                <origin xyz="0.75 1.45 0.9" rpy="0 0 0"/>
                 <geometry>
                     <box size="1.5 0.1 1.5"/>
@@ -43,12 +43,12 @@
             </collision>
             <inertial>
-                <origin xyz="0 0.7 0.825" rpy="0 0 0"/>
+                <origin xyz="0.75 1.45 0.9" rpy="0 0 0"/>
                 <mass value="1"/>
                 <inertia ixx="1" ixy="0" ixz="0" iyy="1" iyz="0" izz="1"/>
             </inertial>
         </link>
-        <link name="wall2">
+        <link name="wall_g">
             <visual>
-                <origin xyz="-0.7 0 0.825" rpy="0 0 0"/>
+                <origin xyz="0.05 0.75 0.9" rpy="0 0 0"/>
                 <geometry>
                     <box size="0.1 1.5 1.5"/>
@@ -59,5 +59,5 @@
             </visual>
             <collision>
-                <origin xyz="-0.7 0 0.825" rpy="0 0 0"/>
+                <origin xyz="0.05 0.75 0.9" rpy="0 0 0"/>
                 <geometry>
                     <box size="0.1 1.5 1.5"/>
@@ -65,12 +65,12 @@
             </collision>
             <inertial>
-                <origin xyz="-0.7 0 0.825" rpy="0 0 0"/>
+                <origin xyz="0.05 0.75 0.9" rpy="0 0 0"/>
                 <mass value="1"/>
                 <inertia ixx="1" ixy="0" ixz="0" iyy="1" iyz="0" izz="1"/>
             </inertial>
         </link>
-        <link name="wall3">
+        <link name="wall_d">
             <visual>
-                <origin xyz="0.7 0 0.825" rpy="0 0 0"/>
+                <origin xyz="1.45 0.75 0.9" rpy="0 0 0"/>
                 <geometry>
                     <box size="0.1 1.5 1.5"/>
@@ -81,5 +81,5 @@
             </visual>
             <collision>
-                <origin xyz="0.7 0 0.825" rpy="0 0 0"/>
+                <origin xyz="1.45 0.75 0.9" rpy="0 0 0"/>
                 <geometry>
                     <box size="0.1 1.5 1.5"/>
@@ -87,5 +87,5 @@
             </collision>
             <inertial>
-                <origin xyz="0.7 0 0.825" rpy="0 0 0"/>
+                <origin xyz="1.45 0.75 0.9" rpy="0 0 0"/>
                 <mass value="1"/>
                 <inertia ixx="1" ixy="0" ixz="0" iyy="1" iyz="0" izz="1"/>
@@ -93,22 +93,20 @@
         </link>
         <!-- joint list pour le socle -->
-        <joint name="box_fixed" type="revolute">
+        <joint name="box_fixed" type="fixed">
             <parent link="world"/>
             <child link="box"/>
-            <origin xyz="0.75 0.75 0.075" rpy="0 0 0" />
-            <dynamics damping="1"/>
-            <limit lower="-3.14159" upper="3.14159" effort="10.0" velocity="0.5"/>
+            <!--origin xyz="0.75 0.75 0.075" rpy="0 0 0" /-->
         </joint>
         <joint name="wall1_fixed" type="fixed">
             <parent link="box"/>
-            <child link="wall1"/>
+            <child link="wall_fond"/>
         </joint>
         <joint name="wall2_fixed" type="fixed">
             <parent link="box"/>
-            <child link="wall2"/>
+            <child link="wall_g"/>
         </joint>
         <joint name="wall3_fixed" type="fixed">
             <parent link="box"/>
-            <child link="wall3"/>
+            <child link="wall_d"/>
         </joint>
     </xacro:macro>

File: src/motoman/motoman_hc10_support/urdf/hc10_gazebo_macro.xacro (robot description, xacro)
@@ -32,7 +32,7 @@
         </xacro:macro>
         <xacro:hc10_env link="${prefix}box_fixed"/>
-        <xacro:hc10_env link="${prefix}wall1"/>
-        <xacro:hc10_env link="${prefix}wall2"/>
-        <xacro:hc10_env link="${prefix}wall3"/>
+        <xacro:hc10_env link="${prefix}wall_fond"/>
+        <xacro:hc10_env link="${prefix}wall_g"/>
+        <xacro:hc10_env link="${prefix}wall_d"/>
         <xacro:hc10_obj link="${prefix}cardboard_box"/>
         <xacro:hc10_arm link="${prefix}base_link"/>

File: src/motoman/motoman_hc10_support/urdf/hc10_objet_macro.xacro (robot description, xacro)
@@ -4,5 +4,5 @@
         <link name="cardboard_box">
             <visual>
-                <origin xyz="0.3 0.15 0.15" rpy="0 0 0"/>
+                <origin xyz="1.05 0.9 0.25" rpy="0 0 0"/>
                 <geometry>
                     <sphere radius="0.1"/>
@@ -13,5 +13,5 @@
             </visual>
             <collision>
-                <origin xyz="0.3 0.15 0.15" rpy="0 0 0"/>
+                <origin xyz="1.05 0.9 0.25" rpy="0 0 0"/>
                 <geometry>
                     <sphere radius="0.1"/>
@@ -19,5 +19,5 @@
             </collision>
             <inertial>
-                <origin xyz="0.3 0.15 0.15" rpy="0 0 0"/>
+                <origin xyz="1.05 0.9 0.25" rpy="0 0 0"/>
                 <mass value="1"/>
                 <inertia ixx="0.01" ixy="0" ixz="0" iyy="0.01" iyz="0" izz="0.01"/>
