Commit message: almost finished advanced trajectory

File: src/motoman/motoman_hc10_support/urdf/hc10_gazebo_macro.xacro (robot description, xacro)
@@ -24,15 +24,8 @@
             </gazebo>
         </xacro:macro>
-        <xacro:macro name="hc10_hand_gazebo" params="link">
-            <gazebo reference="${link}">
-                <material>Gazebo/DarkMagentaTransparent</material>
-                <mu1>0.2</mu1>
-                <mu2>0.2</mu2>
-            </gazebo>
-        </xacro:macro>
         <xacro:hc10_env link="${prefix}box_fixed"/>
-        <xacro:hc10_env link="${prefix}wall1"/>
-        <xacro:hc10_env link="${prefix}wall2"/>
-        <xacro:hc10_env link="${prefix}wall3"/>
+        <xacro:hc10_env link="${prefix}wall_fond"/>
+        <xacro:hc10_env link="${prefix}wall_g"/>
+        <xacro:hc10_env link="${prefix}wall_d"/>
         <xacro:hc10_obj link="${prefix}cardboard_box"/>
         <xacro:hc10_arm link="${prefix}base_link"/>
@@ -42,5 +35,5 @@
         <xacro:hc10_arm link="${prefix}link_4_r"/>
         <xacro:hc10_arm link="${prefix}link_5_b"/>
-        <xacro:hc10_hand_gazebo link="${prefix}link_6_t"/>
+        <xacro:hc10_arm link="${prefix}link_6_t"/>
     </xacro:macro>
 </robot>

File: src/motoman/motoman_hc10_support/urdf/hc10_macro.xacro (robot description, xacro)
@@ -137,5 +137,5 @@
       <parent link="world"/>
       <child link="${prefix}base_link"/>
-      <origin xyz="0.55 0.4 0.15" rpy="0 0 0" />
+      <origin xyz="0.55 0.4 0.16" rpy="0 0 0" />
     </joint>
     <joint name="${prefix}joint_1_s" type="revolute">

File: src/motoman/motoman_hc10_support/urdf/hc10_objet_macro.xacro (robot description, xacro)
@@ -4,5 +4,5 @@
         <link name="cardboard_box">
             <visual>
-                <origin xyz="0.3 0.15 0.15" rpy="0 0 0"/>
+                <origin xyz="1.05 0.9 0.25" rpy="0 0 0"/>
                 <geometry>
                     <sphere radius="0.1"/>
@@ -13,5 +13,5 @@
             </visual>
             <collision>
-                <origin xyz="0.3 0.15 0.15" rpy="0 0 0"/>
+                <origin xyz="1.05 0.9 0.25" rpy="0 0 0"/>
                 <geometry>
                     <sphere radius="0.1"/>
@@ -19,5 +19,5 @@
             </collision>
             <inertial>
-                <origin xyz="0.3 0.15 0.15" rpy="0 0 0"/>
+                <origin xyz="1.05 0.9 0.25" rpy="0 0 0"/>
                 <mass value="1"/>
                 <inertia ixx="0.01" ixy="0" ixz="0" iyy="0.01" iyz="0" izz="0.01"/>
