Commit message: merge capteur into main

File: src/motoman/motoman_hc10_support/urdf/hc10.xacro (robot description, xacro)
@@ -2,4 +2,6 @@
 <robot name="motoman_hc10" xmlns:xacro="http://ros.org/wiki/xacro">
   <xacro:include filename="$(find motoman_hc10_support)/urdf/hc10_macro.xacro" />
+  <xacro:include filename="$(find motoman_hc10_support)/urdf/hc10_sensor.xacro" />
   <xacro:motoman_hc10 prefix=""/>
+  <xacro:motoman_hc10_sensor prefix=""/>
 </robot>

File: src/motoman/motoman_hc10_support/urdf/hc10_macro.xacro (robot description, xacro)
@@ -28,9 +28,4 @@
     </link>
     <link name="${prefix}link_1_s">
-      <inertial>
-        <origin xyz="0 0 0" rpy="0 0 0"/>
-        <mass value="0.1"/>
-        <inertia ixx="0.03" ixy="0.03" ixz="0.03" iyy="0.0" iyz="0.0" izz="0.0"/>
-      </inertial>
       <visual>
         <geometry>
@@ -46,9 +41,4 @@
     </link>
     <link name="${prefix}link_2_l">
-      <inertial>
-        <origin xyz="0 0 0" rpy="0 0 0"/>
-        <mass value="0.1"/>
-        <inertia ixx="0.03" ixy="0.03" ixz="0.03" iyy="0.0" iyz="0.0" izz="0.0"/>
-      </inertial>
       <visual>
         <geometry>
@@ -61,12 +51,7 @@
           <mesh filename="package://motoman_hc10_support/meshes/hc10/collision/link_2_l.stl"/>
         </geometry>
-      </collision>hc10_macro
+      </collision>
     </link>
     <link name="${prefix}link_3_u">
-      <inertial>
-        <origin xyz="0 0 0" rpy="0 0 0"/>
-        <mass value="0.1"/>
-        <inertia ixx="0.03" ixy="0.03" ixz="0.03" iyy="0.0" iyz="0.0" izz="0.0"/>
-      </inertial>
       <visual>
         <geometry>
@@ -82,9 +67,4 @@
     </link>
     <link name="${prefix}link_4_r">
-      <inertial>
-        <origin xyz="0 0 0" rpy="0 0 0"/>
-        <mass value="0.1"/>
-        <inertia ixx="0.03" ixy="0.03" ixz="0.03" iyy="0.0" iyz="0.0" izz="0.0"/>
-      </inertial>
       <visual>
         <geometry>
@@ -100,9 +80,4 @@
     </link>
     <link name="${prefix}link_5_b">
-      <inertial>
-        <origin xyz="0 0 0" rpy="0 0 0"/>
-        <mass value="0.1"/>
-        <inertia ixx="0.03" ixy="0.03" ixz="0.03" iyy="0.0" iyz="0.0" izz="0.0"/>
-      </inertial>
       <visual>
         <geometry>
@@ -118,9 +93,4 @@
     </link>
     <link name="${prefix}link_6_t">
-      <inertial>
-        <origin xyz="0 0 0" rpy="0 0 0"/>
-        <mass value="0.1"/>
-        <inertia ixx="0.03" ixy="0.03" ixz="0.03" iyy="0.0" iyz="0.0" izz="0.0"/>
-      </inertial>
       <visual>
         <geometry>

Commit message: modified environment

File: src/motoman/motoman_hc10_support/urdf/hc10.xacro (robot description, xacro)
@@ -4,6 +4,8 @@
   <xacro:include filename="$(find motoman_hc10_support)/urdf/hc10_gazebo_macro.xacro"/>
   <xacro:include filename="$(find motoman_hc10_support)/urdf/hc10_control.xacro"/>
+  <xacro:include filename="$(find motoman_hc10_support)/urdf/hc10_env_macro.xacro"/>
   <xacro:motoman_hc10 prefix=""/>
   <xacro:hc10_gazebo prefix=""/>
   <xacro:hc10_control prefix=""/>
+  <xacro:hc10_workspace prefix=""/>
 </robot>

File: src/motoman/motoman_hc10_support/urdf/hc10_env_macro.xacro (robot description, xacro)
@@ -7,5 +7,5 @@
               <origin xyz="0 0 0" rpy="0 0 0"/>
               <geometry>
-                <box size="1 1 1"/>
+                <box size="1.5 1.5 0.15"/>
              </geometry>
               <material name="blue">
@@ -16,5 +16,5 @@
               <origin xyz="0 0 0" rpy="0 0 0"/>
               <geometry>
-                <box size="1 1 1"/>
+                <box size="1.5 1.5 0.15"/>
               </geometry>
             </collision>
@@ -26,7 +26,10 @@
         </link>
         <!-- joint list -->
-        <joint name="box_fixed" type="fixed">
+        <joint name="box_fixed" type="revolute">
             <parent link="world"/>
-            <child link="box"/>
+            <child link="${prefix}box"/>
+            <origin xyz="0.75 0.75 0.075" rpy="0 0 0" />
+            <dynamics damping="1"/>
+            <limit lower="-3.14159" upper="3.14159" effort="10.0" velocity="0.5"/>
         </joint>
     </xacro:macro>

File: src/motoman/motoman_hc10_support/urdf/hc10_gazebo_macro.xacro (robot description, xacro)
@@ -3,5 +3,12 @@
 <robot xmlns:xacro="http://www.ros.org/wiki/xacro">
     <xacro:macro name="hc10_gazebo" params="prefix">
-        <xacro:macro name="hc10_arm_gazebo" params="link">
+        <xacro:macro name="hc10_env" params="link">
+            <gazebo reference="${link}">
+                <material>Gazebo/Blue</material>
+                <mu1>0.2</mu1>
+                <mu2>0.2</mu2>
+            </gazebo>
+        </xacro:macro>
+        <xacro:macro name="hc10_arm" params="link">
             <gazebo reference="${link}">
                 <material>Gazebo/White</material>
@@ -17,10 +24,11 @@
             </gazebo>
         </xacro:macro>
-        <xacro:hc10_arm_gazebo link="${prefix}base_link"/>
-        <xacro:hc10_arm_gazebo link="${prefix}link_1_s"/>
-        <xacro:hc10_arm_gazebo link="${prefix}link_2_l"/>
-        <xacro:hc10_arm_gazebo link="${prefix}link_3_u"/>
-        <xacro:hc10_arm_gazebo link="${prefix}link_4_r"/>
-        <xacro:hc10_arm_gazebo link="${prefix}link_5_b"/>
+        <xacro:hc10_env link="${prefix}box_fixed"/>
+        <xacro:hc10_arm link="${prefix}base_link"/>
+        <xacro:hc10_arm link="${prefix}link_1_s"/>
+        <xacro:hc10_arm link="${prefix}link_2_l"/>
+        <xacro:hc10_arm link="${prefix}link_3_u"/>
+        <xacro:hc10_arm link="${prefix}link_4_r"/>
+        <xacro:hc10_arm link="${prefix}link_5_b"/>
         <xacro:hc10_hand_gazebo link="${prefix}link_6_t"/>
     </xacro:macro>

File: src/motoman/motoman_hc10_support/urdf/hc10_macro.xacro (robot description, xacro)
@@ -137,5 +137,5 @@
       <parent link="world"/>
       <child link="${prefix}base_link"/>
-      <origin xyz="0 0 0.5" rpy="0 0 0" />
+      <origin xyz="0.1 0.1 0.5" rpy="0 0 0" />
     </joint>
     <joint name="${prefix}joint_1_s" type="revolute">

Commit message: Setup camera + correction setup

File: src/motoman/motoman_hc10_support/urdf/hc10.xacro (robot description, xacro)
@@ -2,6 +2,12 @@
 <robot name="motoman_hc10" xmlns:xacro="http://ros.org/wiki/xacro">
   <xacro:include filename="$(find motoman_hc10_support)/urdf/hc10_macro.xacro" />
+  <xacro:include filename="$(find motoman_hc10_support)/urdf/hc10_gazebo_macro.xacro"/>
+  <xacro:include filename="$(find motoman_hc10_support)/urdf/hc10_control.xacro"/>
+  <xacro:include filename="$(find motoman_hc10_support)/urdf/hc10_env_macro.xacro"/>
   <xacro:include filename="$(find motoman_hc10_support)/urdf/hc10_sensor.xacro" />
   <xacro:motoman_hc10 prefix=""/>
+  <xacro:hc10_gazebo prefix=""/>
+  <xacro:hc10_control prefix=""/>
+  <xacro:hc10_workspace prefix=""/>
   <xacro:motoman_hc10_sensor prefix=""/>
 </robot>

File: src/motoman/motoman_hc10_support/urdf/hc10_macro.xacro (robot description, xacro)
@@ -5,107 +5,138 @@
     <!-- link list -->
     <link name="world"/>
+    <link name="${prefix}base_link">
+      <inertial>
+        <origin xyz="0 0 0" rpy="0 0 0"/>
+        <mass value="0.1"/>
+        <inertia ixx="0.03" ixy="0.03" ixz="0.03" iyy="0.0" iyz="0.0" izz="0.0"/>
+      </inertial>
+      <visual>
+        <geometry>
+          <mesh filename="package://motoman_hc10_support/meshes/hc10/visual/base_link.dae"/>
+        </geometry>
+        <xacro:material_yaskawa_blue/>
+      </visual>
+      <collision>
+        <geometry>
+          <mesh filename="package://motoman_hc10_support/meshes/hc10/collision/base_link.stl"/>
+        </geometry>
+      </collision>
+    </link>
+    <link name="${prefix}link_1_s">
+      <inertial>
+        <origin xyz="0 0 0" rpy="0 0 0"/>
+        <mass value="0.1"/>
+        <inertia ixx="0.03" ixy="0.03" ixz="0.03" iyy="0.0" iyz="0.0" izz="0.0"/>
+      </inertial>
+      <visual>
+        <geometry>
+          <mesh filename="package://motoman_hc10_support/meshes/hc10/visual/link_1_s.dae"/>
+        </geometry>
+        <xacro:material_yaskawa_blue/>
+      </visual>
+      <collision>
+        <geometry>
+          <mesh filename="package://motoman_hc10_support/meshes/hc10/collision/link_1_s.stl"/>
+        </geometry>
+      </collision>
+    </link>
+    <link name="${prefix}link_2_l">
+      <inertial>
+        <origin xyz="0 0 0" rpy="0 0 0"/>
+        <mass value="0.1"/>
+        <inertia ixx="0.03" ixy="0.03" ixz="0.03" iyy="0.0" iyz="0.0" izz="0.0"/>
+      </inertial>
+      <visual>
+        <geometry>
+          <mesh filename="package://motoman_hc10_support/meshes/hc10/visual/link_2_l.dae"/>
+        </geometry>
+        <xacro:material_yaskawa_blue/>
+      </visual>
+      <collision>
+        <geometry>
+          <mesh filename="package://motoman_hc10_support/meshes/hc10/collision/link_2_l.stl"/>
+        </geometry>
+      </collision>hc10_macro
+    </link>
+    <link name="${prefix}link_3_u">
+      <inertial>
+        <origin xyz="0 0 0" rpy="0 0 0"/>
+        <mass value="0.1"/>
+        <inertia ixx="0.03" ixy="0.03" ixz="0.03" iyy="0.0" iyz="0.0" izz="0.0"/>
+      </inertial>
+      <visual>
+        <geometry>
+          <mesh filename="package://motoman_hc10_support/meshes/hc10/visual/link_3_u.dae"/>
+        </geometry>
+        <xacro:material_yaskawa_blue/>
+      </visual>
+      <collision>
+        <geometry>
+          <mesh filename="package://motoman_hc10_support/meshes/hc10/collision/link_3_u.stl"/>
+        </geometry>
+      </collision>
+    </link>
+    <link name="${prefix}link_4_r">
+      <inertial>
+        <origin xyz="0 0 0" rpy="0 0 0"/>
+        <mass value="0.1"/>
+        <inertia ixx="0.03" ixy="0.03" ixz="0.03" iyy="0.0" iyz="0.0" izz="0.0"/>
+      </inertial>
+      <visual>
+        <geometry>
+          <mesh filename="package://motoman_hc10_support/meshes/hc10/visual/link_4_r.dae"/>
+        </geometry>
+        <xacro:material_yaskawa_blue/>
+      </visual>
+      <collision>
+        <geometry>
+          <mesh filename="package://motoman_hc10_support/meshes/hc10/collision/link_4_r.stl"/>
+        </geometry>
+      </collision>
+    </link>
+    <link name="${prefix}link_5_b">
+      <inertial>
+        <origin xyz="0 0 0" rpy="0 0 0"/>
+        <mass value="0.1"/>
+        <inertia ixx="0.03" ixy="0.03" ixz="0.03" iyy="0.0" iyz="0.0" izz="0.0"/>
+      </inertial>
+      <visual>
+        <geometry>
+          <mesh filename="package://motoman_hc10_support/meshes/hc10/visual/link_5_b.dae"/>
+        </geometry>
+        <xacro:material_yaskawa_blue/>
+      </visual>
+      <collision>
+        <geometry>
+          <mesh filename="package://motoman_hc10_support/meshes/hc10/collision/link_5_b.stl"/>
+        </geometry>
+      </collision>
+    </link>
+    <link name="${prefix}link_6_t">
+      <inertial>
+        <origin xyz="0 0 0" rpy="0 0 0"/>
+        <mass value="0.1"/>
+        <inertia ixx="0.03" ixy="0.03" ixz="0.03" iyy="0.0" iyz="0.0" izz="0.0"/>
+      </inertial>
+      <visual>
+        <geometry>
+          <mesh filename="package://motoman_hc10_support/meshes/hc10/visual/link_6_t.dae"/>
+        </geometry>
+        <xacro:material_yaskawa_blue/>
+      </visual>
+      <collision>
+        <geometry>
+          <mesh filename="package://motoman_hc10_support/meshes/hc10/collision/link_6_t.stl"/>
+        </geometry>
+      </collision>
+    </link>
+    <link name="${prefix}tool0"/>
+    <!-- end of link list -->
+    <!-- joint list -->
     <joint name="world_fixed" type="fixed">
       <parent link="world"/>
       <child link="${prefix}base_link"/>
-    </joint>
-    <link name="${prefix}base_link">
-      <inertial>
-        <origin xyz="0 0 0" rpy="0 0 0"/>
-        <mass value="0.1"/>
-        <inertia ixx="0.03" ixy="0.03" ixz="0.03" iyy="0.0" iyz="0.0" izz="0.0"/>
-      </inertial>
-      <visual>
-        <geometry>
-          <mesh filename="package://motoman_hc10_support/meshes/hc10/visual/base_link.dae"/>
-        </geometry>
-        <xacro:material_yaskawa_blue/>
-      </visual>
-      <collision>
-        <geometry>
-          <mesh filename="package://motoman_hc10_support/meshes/hc10/collision/base_link.stl"/>
-        </geometry>
-      </collision>
-    </link>
-    <link name="${prefix}link_1_s">
-      <visual>
-        <geometry>
-          <mesh filename="package://motoman_hc10_support/meshes/hc10/visual/link_1_s.dae"/>
-        </geometry>
-        <xacro:material_yaskawa_blue/>
-      </visual>
-      <collision>
-        <geometry>
-          <mesh filename="package://motoman_hc10_support/meshes/hc10/collision/link_1_s.stl"/>
-        </geometry>
-      </collision>
-    </link>
-    <link name="${prefix}link_2_l">
-      <visual>
-        <geometry>
-          <mesh filename="package://motoman_hc10_support/meshes/hc10/visual/link_2_l.dae"/>
-        </geometry>
-        <xacro:material_yaskawa_blue/>
-      </visual>
-      <collision>
-        <geometry>
-          <mesh filename="package://motoman_hc10_support/meshes/hc10/collision/link_2_l.stl"/>
-        </geometry>
-      </collision>
-    </link>
-    <link name="${prefix}link_3_u">
-      <visual>
-        <geometry>
-          <mesh filename="package://motoman_hc10_support/meshes/hc10/visual/link_3_u.dae"/>
-        </geometry>
-        <xacro:material_yaskawa_blue/>
-      </visual>
-      <collision>
-        <geometry>
-          <mesh filename="package://motoman_hc10_support/meshes/hc10/collision/link_3_u.stl"/>
-        </geometry>
-      </collision>
-    </link>
-    <link name="${prefix}link_4_r">
-      <visual>
-        <geometry>
-          <mesh filename="package://motoman_hc10_support/meshes/hc10/visual/link_4_r.dae"/>
-        </geometry>
-        <xacro:material_yaskawa_blue/>
-      </visual>
-      <collision>
-        <geometry>
-          <mesh filename="package://motoman_hc10_support/meshes/hc10/collision/link_4_r.stl"/>
-        </geometry>
-      </collision>
-    </link>
-    <link name="${prefix}link_5_b">
-      <visual>
-        <geometry>
-          <mesh filename="package://motoman_hc10_support/meshes/hc10/visual/link_5_b.dae"/>
-        </geometry>
-        <xacro:material_yaskawa_blue/>
-      </visual>
-      <collision>
-        <geometry>
-          <mesh filename="package://motoman_hc10_support/meshes/hc10/collision/link_5_b.stl"/>
-        </geometry>
-      </collision>
-    </link>
-    <link name="${prefix}link_6_t">
-      <visual>
-        <geometry>
-          <mesh filename="package://motoman_hc10_support/meshes/hc10/visual/link_6_t.dae"/>
-        </geometry>
-        <xacro:material_yaskawa_blue/>
-      </visual>
-      <collision>
-        <geometry>
-          <mesh filename="package://motoman_hc10_support/meshes/hc10/collision/link_6_t.stl"/>
-        </geometry>
-      </collision>
-    </link>
-    <link name="${prefix}tool0"/>
-    <!-- end of link list -->
-    <!-- joint list -->
+      <origin xyz="0.1 0.1 0.5" rpy="0 0 0" />
+    </joint>
     <joint name="${prefix}joint_1_s" type="revolute">
       <parent link="${prefix}base_link"/>

File: src/motoman/motoman_hc10_support/urdf/hc10_sensor.xacro (robot description, xacro)
@@ -20,4 +20,40 @@
      </visual>
    </link>
+   <gazebo reference="${prefix}camera_link">
+    <sensor name="kinect_camera" type="depth">
+        <update_rate>20</update_rate>
+        <camera>
+            <horizontal_fov>1.047198</horizontal_fov>
+            <image>
+                <width>640</width>
+                <height>480</height>
+                <format>B8G8R8</format>
+            </image>
+            <clip>
+                <near>0.05</near>
+                <far>3</far>
+            </clip>
+        </camera>
+        <plugin name="kinect_controller" filename="libgazebo_ros_openni_kinect.so">
+        <baseline>0.1</baseline>
+        <alwaysOn>true</alwaysOn>
+        <updateRate>10</updateRate>
+        <cameraName>camera_ir</cameraName>
+        <imageTopicName>/camera/color/image_raw</imageTopicName>
+        <cameraInfoTopicName>/camera/color/camera_info</cameraInfoTopicName>
+        <depthImageTopicName>/camera/depth/image_raw</depthImageTopicName>
+        <depthImageCameraInfoTopicName>/camera/depth/camera_info</depthImageCameraInfoTopicName>
+        <pointCloudTopicName>/camera/depth/points</pointCloudTopicName>
+        <frameName>camera_depth_optical_frame</frameName>
+        <distortion_k1>0.0</distortion_k1>
+        <distortion_k2>0.0</distortion_k2>
+        <distortion_k3>0.0</distortion_k3>
+        <distortion_t1>0.0</distortion_t1>
+        <distortion_t2>0.0</distortion_t2>
+        <pointCloudCutoff>0.16</pointCloudCutoff>
+        <pointCloudCutoffMax>10.0</pointCloudCutoffMax>
+        </plugin>
+    </sensor>
+</gazebo>
     <!-- end of joint list -->
   </xacro:macro>

Commit message: finished env

File: src/motoman/motoman_hc10_support/urdf/hc10.xacro (robot description, xacro)
@@ -5,7 +5,9 @@
   <xacro:include filename="$(find motoman_hc10_support)/urdf/hc10_control.xacro"/>
   <xacro:include filename="$(find motoman_hc10_support)/urdf/hc10_env_macro.xacro"/>
+  <xacro:include filename="$(find motoman_hc10_support)/urdf/hc10_objet_macro.xacro"/>
   <xacro:motoman_hc10 prefix=""/>
   <xacro:hc10_gazebo prefix=""/>
   <xacro:hc10_control prefix=""/>
   <xacro:hc10_workspace prefix=""/>
+  <xacro:hc10_cardboard prefix=""/>
 </robot>

File: src/motoman/motoman_hc10_support/urdf/hc10_env_macro.xacro (robot description, xacro)
@@ -10,5 +10,5 @@
                 </geometry>
                 <material name="blue">
-                    <color rgba="0 0 0.8 1"/>
+                    <color rgba="0.114 0.122 0.102 1"/>
                 </material>
             </visual>

File: src/motoman/motoman_hc10_support/urdf/hc10_gazebo_macro.xacro (robot description, xacro)
@@ -5,5 +5,12 @@
         <xacro:macro name="hc10_env" params="link">
             <gazebo reference="${link}">
-                <material>Gazebo/Blue</material>
+                <material>Gazebo/Pedestrian</material>
+                <mu1>0.2</mu1>
+                <mu2>0.2</mu2>
+            </gazebo>
+        </xacro:macro>
+        <xacro:macro name="hc10_obj" params="link">
+            <gazebo reference="${link}">
+                <material>Gazebo/WoodFloor </material>
                 <mu1>0.2</mu1>
                 <mu2>0.2</mu2>
@@ -12,5 +19,5 @@
         <xacro:macro name="hc10_arm" params="link">
             <gazebo reference="${link}">
-                <material>Gazebo/White</material>
+                <material>Gazebo/White </material>
                 <mu1>0.2</mu1>
                 <mu2>0.2</mu2>
@@ -19,5 +26,5 @@
         <xacro:macro name="hc10_hand_gazebo" params="link">
             <gazebo reference="${link}">
-                <material>Gazebo/Grey</material>
+                <material>Gazebo/DarkMagentaTransparent</material>
                 <mu1>0.2</mu1>
                 <mu2>0.2</mu2>
@@ -28,4 +35,5 @@
         <xacro:hc10_env link="${prefix}wall2"/>
         <xacro:hc10_env link="${prefix}wall3"/>
+        <xacro:hc10_obj link="${prefix}cardboard_box"/>
         <xacro:hc10_arm link="${prefix}base_link"/>
         <xacro:hc10_arm link="${prefix}link_1_s"/>

File: src/motoman/motoman_hc10_support/urdf/hc10_macro.xacro (robot description, xacro)
@@ -193,11 +193,4 @@
     </joint>
     <!-- end of joint list -->
-    <!-- ROS base_link to Robot Manufacturer World Coordinates transform -->
-    <link name="${prefix}base" />
-    <joint name="${prefix}base_link-base" type="fixed">
-      <origin xyz="0 0 0.275" rpy="0 0 0"/>
-      <parent link="${prefix}base_link"/>
-      <child link="${prefix}base"/>
-    </joint>
   </xacro:macro>
 </robot>

Commit message: end

File: src/motoman/motoman_hc10_support/urdf/hc10.xacro (robot description, xacro)
@@ -4,10 +4,10 @@
   <xacro:include filename="$(find motoman_hc10_support)/urdf/hc10_gazebo_macro.xacro"/>
   <xacro:include filename="$(find motoman_hc10_support)/urdf/hc10_control.xacro"/>
-  <xacro:include filename="$(find motoman_hc10_support)/urdf/hc10_env_macro.xacro"/>
+  <!--xacro:include filename="$(find motoman_hc10_support)/urdf/hc10_env_macro.xacro"/-->
   <xacro:include filename="$(find motoman_hc10_support)/urdf/hc10_sensor.xacro" />
   <xacro:motoman_hc10 prefix=""/>
   <xacro:hc10_gazebo prefix=""/>
   <xacro:hc10_control prefix=""/>
-  <xacro:hc10_workspace prefix=""/>
+  <!--xacro:hc10_workspace prefix=""/-->
   <xacro:motoman_hc10_sensor prefix=""/>
 </robot>

File: src/motoman/motoman_hc10_support/urdf/hc10_sensor.xacro (robot description, xacro)
@@ -5,5 +5,5 @@
     <!-- Attach Kinect -->
     <joint type="fixed" name="camera_joint">
-    	<origin xyz="0 0 0" rpy="0 0 0"/>
+    	<origin xyz="0 0 0.05" rpy="0 0 0"/>
     	<child link="${prefix}camera_link"/>
     	<parent link="${prefix}tool0"/>
